Commit message: renamed root frame to base_link for visualization in RViz

File: src/robot_description/urdf/dual_arm_satellite.urdf (robot description, URDF)
Before this commit: robot dual_arm_satellite, 12 links, 11 joints
Links:
- removed link satellite_bus
- added link base_link, mass 80.0; collision cylinder length=0.06 radius=0.35; visual cylinder length=0.06 radius=0.35
Joints:
- removed joint world_to_bus
- added joint world_to_base_link: type fixed, parent world, child base_link, origin xyz=0 0 0 rpy=0 0 0
- joint left_joint1: parent satellite_bus -> base_link
- joint right_joint1: parent satellite_bus -> base_link

Commit message: shoulder joints now rotating about y axis

File: src/robot_description/urdf/dual_arm_satellite.urdf (robot description, URDF)
Before this commit: robot dual_arm_satellite, 12 links, 11 joints
Links:
- link base_link: geometry collision cylinder length=0.25 radius=0.35; visual cylinder length=0.25 radius=0.35
Joints:
- joint left_joint1: axis 0 0 1 -> 0 1 0; limit lower=-3.14 upper=3.14 effort=0 velocity=10 -> lower=-1.57079632679 upper=1.57079632679 effort=0 velocity=10
- joint right_joint1: axis 0 0 1 -> 0 1 0; limit lower=-3.14 upper=3.14 effort=0 velocity=10 -> lower=-1.57079632679 upper=1.57079632679 effort=0 velocity=10

Commit message: reverted shoulder limits

File: src/robot_description/urdf/dual_arm_satellite.urdf (robot description, URDF)
Before this commit: robot dual_arm_satellite, 12 links, 11 joints
Joints:
- joint left_joint1: limit lower=-1.57079632679 upper=1.57079632679 effort=0 velocity=10 -> lower=-3.14 upper=3.14 effort=0 velocity=10
- joint right_joint1: limit lower=-1.57079632679 upper=1.57079632679 effort=0 velocity=10 -> lower=-3.14 upper=3.14 effort=0 velocity=10

Commit message: joint4 now revolute about x axis and limits bumped up to 2pi

File: src/robot_description/urdf/dual_arm_satellite.urdf (robot description, URDF)
Before this commit: robot dual_arm_satellite, 12 links, 11 joints
Joints:
- joint left_joint4: axis 0 0 1 -> 1 0 0; limit lower=-3.14 upper=3.14 effort=0 velocity=10 -> lower=-6.283 upper=6.283 effort=0 velocity=10
- joint right_joint4: axis 0 0 1 -> 1 0 0; limit lower=-3.14 upper=3.14 effort=0 velocity=10 -> lower=-6.283 upper=6.283 effort=0 velocity=10

Commit message: shoulder joints now aligned radially outwards from base

File: src/robot_description/urdf/dual_arm_satellite.urdf (robot description, URDF)
Before this commit: robot dual_arm_satellite, 12 links, 11 joints
Joints:
- joint left_joint2: axis 0 1 0 -> 0 0 1; origin xyz=0.15 0 0 rpy=0 0 0 -> xyz=0 0.15 0 rpy=0 0 0
- joint right_joint2: axis 0 1 0 -> 0 0 1; origin xyz=0.15 0 0 rpy=0 0 0 -> xyz=0 0.15 0 rpy=0 0 0

Commit message: reorient thruster so x-axis is coplanar with rotating direction of j4

File: src/robot_description/urdf/dual_arm_satellite.urdf (robot description, URDF)
Before this commit: robot dual_arm_satellite, 12 links, 11 joints
Joints:
- joint left_ee_fixed: origin xyz=0.12 0 0 rpy=0 0 0 -> xyz=0 0.12 0 rpy=0 0 0
- joint right_ee_fixed: origin xyz=0.12 0 0 rpy=0 0 0 -> xyz=0 0.12 0 rpy=0 0 0

Commit message: fixed origin of link4

File: src/robot_description/urdf/dual_arm_satellite.urdf (robot description, URDF)
Before this commit: robot dual_arm_satellite, 12 links, 11 joints
Joints:
- joint right_joint4: origin xyz=0.30 0 0 rpy=0 0 0 -> xyz=0.0 0 0 rpy=0 0 0

Commit message: fixed end-effector frame to align with +x face of link4

File: src/robot_description/urdf/dual_arm_satellite.urdf (robot description, URDF)
Before this commit: robot dual_arm_satellite, 12 links, 11 joints
Joints:
- joint left_ee_fixed: origin xyz=0 0.12 0 rpy=0 0 0 -> xyz=0 0.06 0 rpy=0 0 0
- joint right_ee_fixed: origin xyz=0 0.12 0 rpy=0 0 0 -> xyz=0 0.06 0 rpy=0 0 0
- joint right_joint4: origin xyz=0.0 0 0 rpy=0 0 0 -> xyz=0.30 0 0 rpy=0 0 0

Commit message: fixed joint 2 limits and orientation

File: src/robot_description/urdf/dual_arm_satellite.urdf (robot description, URDF)
Before this commit: robot dual_arm_satellite, 12 links, 11 joints
Joints:
- joint left_joint3: origin xyz=0.35 0 0 rpy=0 0 0 -> xyz=0 0.35 0 rpy=0 0 0
- joint right_joint3: origin xyz=0.35 0 0 rpy=0 0 0 -> xyz=0 0.35 0 rpy=0 0 0

Commit message: now joint 2 limits fixed

File: src/robot_description/urdf/dual_arm_satellite.urdf (robot description, URDF)
Before this commit: robot dual_arm_satellite, 12 links, 11 joints
Joints:
- joint left_joint2: limit lower=-3.14 upper=3.14 effort=0 velocity=10 -> lower=-1.57079 upper=1.57079 effort=0 velocity=10
- joint right_joint2: limit lower=-3.14 upper=3.14 effort=0 velocity=10 -> lower=-1.57079 upper=1.57079 effort=0 velocity=10

Commit message: revert thruster change

File: src/robot_description/urdf/dual_arm_satellite.urdf (robot description, URDF)
Before this commit: robot dual_arm_satellite, 12 links, 11 joints
Joints:
- joint left_ee_fixed: origin xyz=0 0.06 0 rpy=0 0 0 -> xyz=0.12 0 0 rpy=0 0 0
- joint right_ee_fixed: origin xyz=0 0.06 0 rpy=0 0 0 -> xyz=0.12 0 0 rpy=0 0 0

Commit message: revert thruster change

File: src/robot_description/urdf/dual_arm_satellite.urdf (robot description, URDF)
Before this commit: robot dual_arm_satellite, 12 links, 11 joints
Joints:
- joint left_ee_fixed: origin xyz=0.12 0 0 rpy=0 0 0 -> xyz=0 0.06 0 rpy=0 0 0
- joint right_ee_fixed: origin xyz=0.12 0 0 rpy=0 0 0 -> xyz=0 0.06 0 rpy=0 0 0
